Commit message: got gazebo and rviz working with ddrive; but odom is mismatched between the two

File: diff_drive/urdf/ddrive.gazebo.xacro (robot description, xacro)
@@ -31,7 +31,10 @@
             <odom_topic>odom</odom_topic>
             <tf_topic>tf</tf_topic>
+            <!-- frame ids -->
+            <frame_id>odom</frame_id>
+            <child_frame_id>base_link</child_frame_id>
         </plugin>
         <plugin name="ignition::gazebo::systems::JointStatePublisher" filename="libignition-gazebo-joint-state-publisher-system.so">
-            <topic>joint_states</topic>
+            <topic>/joint_states</topic>
         </plugin>
     </gazebo>

File: diff_drive/urdf/ddrive.urdf.xacro (robot description, xacro)
@@ -21,11 +21,12 @@
     <!-- the odom link and joint -->
     <!-- displacement in z chosen to mirror that of the robot being spawned in gazebo -->
-    <link name="odom">
-    </link>
-    <joint name="base_joint" type="fixed">
-        <origin xyz="0 0 1" rpy="0 0 0"/>
+    <!-- <link name="odom">
+    </link> -->
+    <!-- <joint name="base_joint" type="fixed">
+        <origin xyz="0 0 0" rpy="0 0 0"/>
         <parent link="odom"/>
         <child link="base_link"/>
     </joint>
+     -->
     <!-- the robot base_link -->
     <link name="base_link">
@@ -55,5 +56,5 @@
     <!-- the l_wheel (left wheel) joint and link -->
     <joint name="l_wheel_joint" type="continuous">
-        <origin xyz="${base_length/4} ${base_width/2} ${base_height/2}" rpy="1.57079632679 0 0"/>
+        <origin xyz="${base_length/4} ${base_width/2} ${base_height/2}" rpy="-1.57079632679 0 0"/>
         <parent link="base_link"/>
         <child link="l_wheel_link"/>
@@ -63,5 +64,5 @@
     <link name="l_wheel_link"   >
         <visual>
-            <origin xyz="0 0 -${wheel_thickness/2}" rpy="0 0 0"/>
+            <origin xyz="0 0 ${wheel_thickness/2}" rpy="0 0 0"/>
             <geometry>
                 <cylinder length="${wheel_thickness}" radius="${wheel_radius}"/>
@@ -72,5 +73,5 @@
         </visual>
         <collision>
-            <origin xyz="0 0 -${wheel_thickness/2}" rpy="0 0 0"/>
+            <origin xyz="0 0 ${wheel_thickness/2}" rpy="0 0 0"/>
             <geometry>
                 <cylinder length="${wheel_thickness}" radius="${wheel_radius}"/>
@@ -87,5 +88,5 @@
     <!-- the r_wheel (right wheel) joint and link -->
     <joint name="r_wheel_joint" type="continuous">
-        <origin xyz="${base_length/4} -${base_width/2} ${base_height/2}" rpy="1.57079632679 0 0"/>
+        <origin xyz="${base_length/4} -${base_width/2} ${base_height/2}" rpy="-1.57079632679 0 0"/>
         <parent link="base_link"/>
         <child link="r_wheel_link"/>
@@ -95,5 +96,5 @@
     <link name="r_wheel_link">
         <visual>
-            <origin xyz="0 0 ${wheel_thickness/2}" rpy="0 0 0"/>
+            <origin xyz="0 0 -${wheel_thickness/2}" rpy="0 0 0"/>
             <geometry>
                 <cylinder length="${wheel_thickness}" radius="${wheel_radius}"/>
@@ -104,5 +105,5 @@
         </visual>
         <collision>
-            <origin xyz="0 0 ${wheel_thickness/2}" rpy="0 0 0"/>
+            <origin xyz="0 0 -${wheel_thickness/2}" rpy="0 0 0"/>
             <geometry>
                 <cylinder length="${wheel_thickness}" radius="${wheel_radius}"/>
