Commit message: started building the robot urdf; still need to add casters

File: diff_drive/urdf/ddrive.urdf.xacro (robot description, xacro)
@@ -4,23 +4,26 @@
     <xacro:property name="yaml_file" value="$(find diff_drive)/config/ddrive.yaml" />
     <xacro:property name="props" value="${xacro.load_yaml(yaml_file)['/**']['ros__parameters']}" />
-    <!-- platform_height is the same as total height of the turtle -->
-    <xacro:property name="platform_height" value="${props['platform_height']}"/>
+    <!-- dimension parameters of robot -->
     <xacro:property name="wheel_radius" value="${props['wheel_radius']}"/>
-    <xacro:property name="platform_radius" value="${props['platform_radius']}"/>
+    <!-- note: the caster is a sphere -->
+    <xacro:property name="caster_radius" value="${props['caster_radius']}"/>
+    <xacro:property name="base_length" value="${props['base_length']}"/>
+    <xacro:property name="base_width" value="${props['base_width']}"/>
+    <xacro:property name="base_height" value="${props['base_height']}"/>
+    <!-- mass parameters of robot -->
+    <xacro:property name="base_mass" value="${props['base_mass']}"/>
+    <xacro:property name="wheel_mass" value="${props['wheel_mass']}"/>
+    <xacro:property name="caster_mass" value="${props['caster_mass']}"/>
     <!-- constant dimensions -->
-    <xacro:property name="base_length" value="0.125"/>
-    <xacro:property name="cylinder_radius" value="${base_length/2}"/>
-    <xacro:property name="stem_radius" value="${base_length/2}"/>
-    <xacro:property name="platform_thickness" value="0.05"/>
-    <xacro:property name="wheel_thickness" value="0.1"/>
-    <!-- dimensions adaptive to parameters -->
+    <xacro:property name="wheel_thickness" value="0.2"/>
+    <!-- variables adaptive to parameters -->
     <xacro:property name="stem_height" value="${wheel_radius}"/>
     <xacro:property name="cylinder_height" value="${platform_height - (wheel_radius + stem_height + base_length + platform_thickness)}"/>
-    <!-- the turtle robot base_link -->
+    <!-- the robot base_link -->
     <link name="base_link">
         <visual>
-            <origin xyz="0 0 ${base_length/2}" rpy="0 0 0"/>
+            <origin xyz="0 0 ${base_height/2}" rpy="0 0 0"/>
             <geometry>
-                <box size="${base_length} ${base_length} ${base_length}" />
+                <box size="${base_length} ${base_width} ${base_height}" />
             </geometry>
             <material name="green">
@@ -29,7 +32,7 @@
         </visual>
         <collision>
-            <origin xyz="0 0 ${base_length/2}" rpy="0 0 0"/>
+            <origin xyz="0 0 ${base_height/2}" rpy="0 0 0"/>
             <geometry>
-                <box size="${base_length} ${base_length} ${base_length}" />
+                <box size="${base_length} ${base_width} ${base_height}" />
             </geometry>
             <material name="green">
@@ -37,92 +40,20 @@
             </material>
         </collision>
+        <inertial>
+            <mass value="${base_mass}"/>
+            <inertia ixx="${(1/12)*(base_mass)*(base_height**2+base_length**2)}" ixy="0.0" ixz="0.0" iyy="${(1/12)*(base_mass)*(base_width**2+base_length**2)}" iyz="0.0" izz="${(1/12)*(base_mass)*(base_width**2+base_height**2)}"/>
+        </inertial>
     </link>
-    <!-- top half of the turtle 'unicycle' -->
-    <joint name="cylinder_joint" type="fixed">
-        <origin xyz="0 0 ${base_length}" rpy="0 0 0"/>
+    <!-- the l_wheel (left wheel) joint and link -->
+    <joint name="l_wheel_joint" type="continuous">
+        <origin xyz="${base_length/4} ${base_width/2} ${base_height/2}" rpy="1.57079632679 0 0"/>
         <parent link="base_link"/>
-        <child link="cylinder_link"/>
-    </joint>
-    <link name="cylinder_link">
-        <visual>
-            <origin xyz="0 0 ${cylinder_height/2}" rpy="0 0 0"/>
-            <geometry>
-                <cylinder length="${cylinder_height}" radius="${cylinder_radius}"/>
-            </geometry>
-            <material name="red">
-                <color rgba="1 0.2 0.2 1"/>
-            </material>
-        </visual>
-        <collision>
-            <origin xyz="0 0 ${cylinder_height/2}" rpy="0 0 0"/>
-            <geometry>
-                <cylinder length="${cylinder_height}" radius="${cylinder_radius}"/>
-            </geometry>
-            <material name="red">
-                <color rgba="1 0.2 0.2 1"/>
-            </material>
-        </collision>
-    </link>
-    <joint name="platform_joint" type="revolute">
-        <origin xyz="0 0 ${cylinder_height}" rpy="0 0 0"/>
-        <parent link="cylinder_link"/>
-        <child link="platform_link"/>
-        <axis xyz="0 1 0"/>
-        <limit effort="1000.0" lower="-0.5" upper="0.5" velocity="0.5"/>
-    </joint>
-    <link name="platform_link">
-        <visual>
-            <origin xyz="0 0 ${platform_thickness/2}" rpy="0 0 0"/>
-            <geometry>
-                <cylinder length="${platform_thickness}" radius="${platform_radius}"/>
-            </geometry>
-            <material name = "blue">
-                <color rgba="0.2 0.2 1 1"/>
-            </material>
-        </visual>
-        <collision>
-            <origin xyz="0 0 ${platform_thickness/2}" rpy="0 0 0"/>
-            <geometry>
-                <cylinder length="${platform_thickness}" radius="${platform_radius}"/>
-            </geometry>
-        </collision>
-    </link>
-    <!-- bottom half of the turtle 'unicycle' -->
-    <joint name="stem_joint" type="continuous">
-        <origin xyz="0 0 0" rpy="0 0 0"/>
-        <parent link="base_link"/>
-        <child link="stem_link"/>
-        <axis xyz="0 0 1"/>
-    </joint>
-    <link name="stem_link">
-        <visual>
-            <origin xyz="0 0 -${stem_height/2}" rpy="0 0 0"/>
-            <geometry>
-                <cylinder length="${stem_height}" radius="${stem_radius}"/>
-            </geometry>
-            <material name="yellow">
-                <color rgba="1 1 0.2 1"/>
-            </material>
-        </visual>
-        <collision>
-            <origin xyz="0 0 -${stem_height/2}" rpy="0 0 0"/>
-            <geometry>
-                <cylinder length="${stem_height}" radius="${stem_radius}"/>
-            </geometry>
-            <material name="yellow">
-                <color rgba="1 1 0.2 1"/>
-            </material>
-        </collision>
-    </link>
-    <joint name="wheel_joint" type="continuous">
-        <origin xyz="0 0 -${wheel_radius}" rpy="1.57079632679 0 0"/>
-        <parent link="stem_link"/>
-        <child link="wheel_link"/>
+        <child link="l_wheel_link"/>
         <axis xyz="0 0 1"/>
         <limit effort="1000.0" velocity="0.5"/>
     </joint>
-    <link name="wheel_link">
+    <link name="l_wheel_link"   >
         <visual>
-            <origin xyz="0 0 0" rpy="0 0 0"/>
+            <origin xyz="0 0 -${wheel_thickness/2}" rpy="0 0 0"/>
             <geometry>
                 <cylinder length="${wheel_thickness}" radius="${wheel_radius}"/>
@@ -133,5 +64,5 @@
         </visual>
         <collision>
-            <origin xyz="0 0 0" rpy="0 0 0"/>
+            <origin xyz="0 0 -${wheel_thickness/2}" rpy="0 0 0"/>
             <geometry>
                 <cylinder length="${wheel_thickness}" radius="${wheel_radius}"/>
@@ -141,4 +72,40 @@
             </material>
         </collision>
+        <inertial>
+            <mass value="${wheel_mass}"/>
+            <inertia ixx="${(1/12)*(wheel_mass)*(3*wheel_radius**2+wheel_thickness**2)}" ixy="0.0" ixz="0.0" iyy="${(1/12)*(wheel_mass)*(3*wheel_radius**2+wheel_thickness**2)}" iyz="0.0" izz="${(1/2)*(wheel_mass)*(wheel_radius**2)}"/>
+        </inertial>
+    </link>
+    <!-- the r_wheel (right wheel) joint and link -->
+    <joint name="r_wheel_joint" type="continuous">
+        <origin xyz="${base_length/4} -${base_width/2} ${base_height/2}" rpy="1.57079632679 0 0"/>
+        <parent link="base_link"/>
+        <child link="r_wheel_link"/>
+        <axis xyz="0 0 1"/>
+        <limit effort="1000.0" velocity="0.5"/>
+    </joint>
+    <link name="r_wheel_link">
+        <visual>
+            <origin xyz="0 0 ${wheel_thickness/2}" rpy="0 0 0"/>
+            <geometry>
+                <cylinder length="${wheel_thickness}" radius="${wheel_radius}"/>
+            </geometry>
+            <material name="orange">
+                <color rgba="1 0.5 0.1 1"/>
+            </material>
+        </visual>
+        <collision>
+            <origin xyz="0 0 ${wheel_thickness/2}" rpy="0 0 0"/>
+            <geometry>
+                <cylinder length="${wheel_thickness}" radius="${wheel_radius}"/>
+            </geometry>
+            <material name="orange">
+                <color rgba="1 0.5 0.1 1"/>
+            </material>
+        </collision>
+        <inertial>
+            <mass value="${wheel_mass}"/>
+            <inertia ixx="${(1/12)*(wheel_mass)*(3*wheel_radius**2+wheel_thickness**2)}" ixy="0.0" ixz="0.0" iyy="${(1/12)*(wheel_mass)*(3*wheel_radius**2+wheel_thickness**2)}" iyz="0.0" izz="${(1/2)*(wheel_mass)*(wheel_radius**2)}"/>
+        </inertial>
     </link>
 </robot>

Commit message: finished urdf! w/ inertia stuff hopefully

File: diff_drive/urdf/ddrive.urdf.xacro (robot description, xacro)
@@ -91,6 +91,6 @@
                 <cylinder length="${wheel_thickness}" radius="${wheel_radius}"/>
             </geometry>
-            <material name="orange">
-                <color rgba="1 0.5 0.1 1"/>
+            <material name="red">
+                <color rgba="1 0.2 0.2 1"/>
             </material>
         </visual>
@@ -100,6 +100,6 @@
                 <cylinder length="${wheel_thickness}" radius="${wheel_radius}"/>
             </geometry>
-            <material name="orange">
-                <color rgba="1 0.5 0.1 1"/>
+            <material name="red">
+                <color rgba="1 0.2 0.2 1"/>
             </material>
         </collision>
@@ -109,3 +109,63 @@
         </inertial>
     </link>
+    <!-- the t_caster (top caster wheel) joint and link -->
+    <joint name="t_caster_joint" type="fixed">
+        <origin xyz="-${2*base_length/5} 0 ${base_height}" rpy="0 0 0"/>
+        <parent link="base_link"/>
+        <child link="t_caster_link"/>
+    </joint>
+    <link name="t_caster_link">
+        <visual>
+            <origin xyz="0 0 ${caster_radius}" rpy="0 0 0"/>
+            <geometry>
+                <sphere radius="${caster_radius}"/>
+            </geometry>
+            <material name = "blue">
+                <color rgba="0.2 0.2 1 1"/>
+            </material>
+        </visual>
+        <collision>
+            <origin xyz="0 0 ${caster_radius}" rpy="0 0 0"/>
+            <geometry>
+                <sphere radius="${caster_radius}"/>
+            </geometry>
+            <material name = "blue">
+                <color rgba="0.2 0.2 1 1"/>
+            </material>
+        </collision>
+        <inertial>
+            <mass value="${caster_mass}"/>
+            <inertia ixx="${(2/5)*(caster_mass)*(caster_radius**2)}" ixy="0.0" ixz="0.0" iyy="${(2/5)*(caster_mass)*(caster_radius**2)}" iyz="0.0" izz="${(2/5)*(caster_mass)*(caster_radius**2)}"/>
+        </inertial>
+    </link>
+    <!-- the b_caster (bottom caster wheel) joint and link -->
+    <joint name="b_caster_joint" type="fixed">
+        <origin xyz="-${2*base_length/5} 0 0" rpy="0 0 0"/>
+        <parent link="base_link"/>
+        <child link="b_caster_link"/>
+    </joint>
+    <link name="b_caster_link">
+        <visual>
+            <origin xyz="0 0 -${caster_radius}" rpy="0 0 0"/>
+            <geometry>
+                <sphere radius="${caster_radius}"/>
+            </geometry>
+            <material name="yellow">
+                <color rgba="1 1 0.2 1"/>
+            </material>
+        </visual>
+        <collision>
+            <origin xyz="0 0 -${caster_radius}" rpy="0 0 0"/>
+            <geometry>
+                <sphere radius="${caster_radius}"/>
+            </geometry>
+            <material name="yellow">
+                <color rgba="1 1 0.2 1"/>
+            </material>
+        </collision>
+        <inertial>
+            <mass value="${caster_mass}"/>
+            <inertia ixx="${(2/5)*(caster_mass)*(caster_radius**2)}" ixy="0.0" ixz="0.0" iyy="${(2/5)*(caster_mass)*(caster_radius**2)}" iyz="0.0" izz="${(2/5)*(caster_mass)*(caster_radius**2)}"/>
+        </inertial>
+    </link>
 </robot>

Commit message: ddrive.launch file seems to work? Need to get the ddrive plugin to work with keyboard teleop

File: diff_drive/urdf/ddrive.urdf.xacro (robot description, xacro)
@@ -1,4 +1,6 @@
 <?xml version="1.0"?>
 <robot xmlns:xacro="http://www.ros.org/wiki/xacro" name="ddrive">
+    <!-- include the gazebo xacro file -->
+    <xacro:include filename="$(find diff_drive)/ddrive.gazebo.xacro" />
     <!-- loading in parameter file -->
     <xacro:property name="yaml_file" value="$(find diff_drive)/config/ddrive.yaml" />
@@ -17,7 +19,13 @@
     <!-- constant dimensions -->
     <xacro:property name="wheel_thickness" value="0.2"/>
-    <!-- variables adaptive to parameters -->
-    <xacro:property name="stem_height" value="${wheel_radius}"/>
-    <xacro:property name="cylinder_height" value="${platform_height - (wheel_radius + stem_height + base_length + platform_thickness)}"/>
+    <!-- the odom link and joint -->
+    <!-- displacement in z chosen to mirror that of the robot being spawned in gazebo -->
+    <link name="odom">
+    </link>
+    <joint name="base_joint" type="fixed">
+        <origin xyz="0 0 1" rpy="0 0 0"/>
+        <parent link="odom"/>
+        <child link="base_link"/>
+    </joint>
     <!-- the robot base_link -->
     <link name="base_link">

Commit message: correctly adjusted the inertia placement of the robot

File: diff_drive/urdf/ddrive.urdf.xacro (robot description, xacro)
@@ -50,6 +50,9 @@
         </collision>
         <inertial>
+            <origin xyz="0 0 ${base_height/2}" rpy="0 0 0"/>
             <mass value="${base_mass}"/>
-            <inertia ixx="${(1/12)*(base_mass)*(base_height**2+base_length**2)}" ixy="0.0" ixz="0.0" iyy="${(1/12)*(base_mass)*(base_width**2+base_length**2)}" iyz="0.0" izz="${(1/12)*(base_mass)*(base_width**2+base_height**2)}"/>
+            <inertia ixx="${(1/12)*(base_mass)*(base_width**2+base_height**2)}" ixy="0.0" ixz="0.0" iyy="${(1/12)*(base_mass)*(base_height**2+base_length**2)}" iyz="0.0" izz="${(1/12)*(base_mass)*(base_width**2+base_length**2)}"/>
+            <!-- <inertia ixx="${(1/12)*(base_mass)*(base_width**2+base_length**2)}" ixy="0.0" ixz="0.0" iyy="${(1/12)*(base_mass)*(base_height**2+base_length**2)}" iyz="0.0" izz="${(1/12)*(base_mass)*(base_width**2+base_height**2)}"/> -->
+            <!-- <inertia ixx="${(1/12)*(base_mass)*(base_height**2+base_length**2)}" ixy="0.0" ixz="0.0" iyy="${(1/12)*(base_mass)*(base_width**2+base_length**2)}" iyz="0.0" izz="${(1/12)*(base_mass)*(base_width**2+base_height**2)}"/> -->
         </inertial>
     </link>
@@ -80,6 +83,15 @@
                 <color rgba="1 0.5 0.1 1"/>
             </material>
-        </collision>
-        <inertial>
+            <!-- <surface>
+                <friction>
+                    <ode>
+                        <mu>1.0</mu>
+                        <mu2>0.25</mu2>
+                    </ode>
+                </friction>
+            </surface> -->
+        </collision>
+        <inertial>
+            <origin xyz="0 0 ${wheel_thickness/2}" rpy="0 0 0"/>
             <mass value="${wheel_mass}"/>
             <inertia ixx="${(1/12)*(wheel_mass)*(3*wheel_radius**2+wheel_thickness**2)}" ixy="0.0" ixz="0.0" iyy="${(1/12)*(wheel_mass)*(3*wheel_radius**2+wheel_thickness**2)}" iyz="0.0" izz="${(1/2)*(wheel_mass)*(wheel_radius**2)}"/>
@@ -112,6 +124,15 @@
                 <color rgba="1 0.2 0.2 1"/>
             </material>
-        </collision>
-        <inertial>
+            <!-- <surface>
+                <friction>
+                    <ode>
+                        <mu>1.0</mu>
+                        <mu2>0.25</mu2>
+                    </ode>
+                </friction>
+            </surface> -->
+        </collision>
+        <inertial>
+            <origin xyz="0 0 -${wheel_thickness/2}" rpy="0 0 0"/>
             <mass value="${wheel_mass}"/>
             <inertia ixx="${(1/12)*(wheel_mass)*(3*wheel_radius**2+wheel_thickness**2)}" ixy="0.0" ixz="0.0" iyy="${(1/12)*(wheel_mass)*(3*wheel_radius**2+wheel_thickness**2)}" iyz="0.0" izz="${(1/2)*(wheel_mass)*(wheel_radius**2)}"/>
@@ -145,5 +166,5 @@
                 <friction>
                     <ode>
-                        <mu>0.0</mu>
+                        <mu1>0.0</mu1>
                         <mu2>0.0</mu2>
                     </ode>
@@ -152,4 +173,5 @@
         </collision>
         <inertial>
+            <origin xyz="0 0 ${caster_radius}" rpy="0 0 0"/>
             <mass value="${caster_mass}"/>
             <inertia ixx="${(2/5)*(caster_mass)*(caster_radius**2)}" ixy="0.0" ixz="0.0" iyy="${(2/5)*(caster_mass)*(caster_radius**2)}" iyz="0.0" izz="${(2/5)*(caster_mass)*(caster_radius**2)}"/>
@@ -183,5 +205,5 @@
                 <friction>
                     <ode>
-                        <mu>0.0</mu>
+                        <mu1>0.0</mu1>
                         <mu2>0.0</mu2>
                     </ode>
@@ -190,4 +212,5 @@
         </collision>
         <inertial>
+            <origin xyz="0 0 -${caster_radius}" rpy="0 0 0"/>
             <mass value="${caster_mass}"/>
             <inertia ixx="${(2/5)*(caster_mass)*(caster_radius**2)}" ixy="0.0" ixz="0.0" iyy="${(2/5)*(caster_mass)*(caster_radius**2)}" iyz="0.0" izz="${(2/5)*(caster_mass)*(caster_radius**2)}"/>

Commit message: got the flip to work properlygit add .!

File: diff_drive/urdf/ddrive.urdf.xacro (robot description, xacro)
@@ -17,6 +17,7 @@
     <xacro:property name="wheel_mass" value="${props['wheel_mass']}"/>
     <xacro:property name="caster_mass" value="${props['caster_mass']}"/>
+    <xacro:property name="wheel_thickness" value="${props['wheel_thickness']}"/>
     <!-- constant dimensions -->
-    <xacro:property name="wheel_thickness" value="0.2"/>
+    <!-- <xacro:property name="wheel_thickness" value="0.2"/> -->
     <!-- the odom link and joint -->
     <!-- displacement in z chosen to mirror that of the robot being spawned in gazebo -->
@@ -53,6 +54,4 @@
             <mass value="${base_mass}"/>
             <inertia ixx="${(1/12)*(base_mass)*(base_width**2+base_height**2)}" ixy="0.0" ixz="0.0" iyy="${(1/12)*(base_mass)*(base_height**2+base_length**2)}" iyz="0.0" izz="${(1/12)*(base_mass)*(base_width**2+base_length**2)}"/>
-            <!-- <inertia ixx="${(1/12)*(base_mass)*(base_width**2+base_length**2)}" ixy="0.0" ixz="0.0" iyy="${(1/12)*(base_mass)*(base_height**2+base_length**2)}" iyz="0.0" izz="${(1/12)*(base_mass)*(base_width**2+base_height**2)}"/> -->
-            <!-- <inertia ixx="${(1/12)*(base_mass)*(base_height**2+base_length**2)}" ixy="0.0" ixz="0.0" iyy="${(1/12)*(base_mass)*(base_width**2+base_length**2)}" iyz="0.0" izz="${(1/12)*(base_mass)*(base_width**2+base_height**2)}"/> -->
         </inertial>
     </link>
@@ -63,5 +62,5 @@
         <child link="l_wheel_link"/>
         <axis xyz="0 0 1"/>
-        <limit effort="1000.0" velocity="0.5"/>
+        <limit effort="1000.0" velocity="1000.0"/>
     </joint>
     <link name="l_wheel_link"   >
@@ -104,5 +103,5 @@
         <child link="r_wheel_link"/>
         <axis xyz="0 0 1"/>
-        <limit effort="1000.0" velocity="0.5"/>
+        <limit effort="1000.0" velocity="1000.0"/>
     </joint>
     <link name="r_wheel_link">
